File: elec/PCB/CardPCB/CardPCB.kicad_sch (KiCad schematic)
At the start: 20 parts, among them Q1 SL2312, Q2 SL2301S, SW1 SW_DPDT_x2, U1 LM555xM

Commit message: Final PCB
Generation of gerber and sending command
Parts:
- removed D1: TVS 5VWM 14VC SOD323, Diode_THT:D_DO-201AE_P15.24mm_Horizontal, symbol Diode:1N630xCA
Other:
- note added: "TVS diode removed : to big to fit"
Changed lines of the file:
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@@
+		)
+	)
+	(text "TVS diode removed :\nto big to fit\n"
+		(exclude_from_sim no)
+		(at 62.484 34.036 0)
+		(effects
+			(font
+				(size 1.27 1.27)
+			)
 		)
 	)
@@
 	)
 	(junction
-		(at 50.8 27.94)
-		(diameter 0)
-		(color 0 0 0 0)
-	)
-	(junction
 		(at 120.65 27.94)
 		(diameter 0)
@@
 	(wire
 		(pts
-			(xy 50.8 39.37) (xy 50.8 40.64)
-		)
-		(stroke
-			(width 0)
-			(type default)
-		)
-	)
-	(wire
-		(pts
 			(xy 87.63 83.82) (xy 92.71 83.82)
 		)
@@
 	(wire
 		(pts
-			(xy 50.8 27.94) (xy 45.72 27.94)
+			(xy 45.72 27.94) (xy 85.09 27.94)
 		)
 		(stroke
@@
 	(wire
 		(pts
-			(xy 50.8 31.75) (xy 50.8 27.94)
-		)
-		(stroke
-			(width 0)
-			(type default)
-		)
-	)
-	(wire
-		(pts
 			(xy 44.45 153.67) (xy 44.45 157.48)
 		)
@@
 		(pts
 			(xy 87.63 97.79) (xy 87.63 100.33)
-		)
-		(stroke
-			(width 0)
-			(type default)
-		)
-	)
-	(wire
-		(pts
-			(xy 50.8 27.94) (xy 85.09 27.94)
 		)
 		(stroke
@@
 	)
 	(symbol
-		(lib_id "Diode:1N630xCA")
-		(at 50.8 35.56 90)
-		(unit 1)
-		(exclude_from_sim no)
-		(in_bom yes)
-		(on_board yes)
-		(dnp no)
-		(property "Reference" "D1"
-			(at 53.34 34.2899 90)
-			(effects
-				(font
-					(size 1.27 1.27)
-				)
-				(justify right)
-			)
-		)
-		(property "Value" "TVS 5VWM 14VC SOD323"
-			(at 53.34 37.084 90)
-			(effects
-				(font
-					(size 1.27 1.27)
-				)
-				(justify right)
-			)
-		)
-		(property "Footprint" "Diode_THT:D_DO-201AE_P15.24mm_Horizontal"
-			(at 55.88 35.56 0)
-			(effects
-				(font
-					(size 1.27 1.27)
-				)
-				(hide yes)
-			)
-		)
-		(property "Datasheet" "https://www.digikey.ca/en/products/detail/diodes-incorporated/DESD5V0S1BA-7/3451477"
-			(at 50.8 35.56 0)
-			(effects
-				(font
-					(size 1.27 1.27)
-				)
-				(hide yes)
-			)
-		)
-		(property "Description" "1500W bidirectional TRANSZORB® Transient Voltage Suppressor, DO-201AE"
-			(at 50.8 35.56 0)
-			(effects
-				(font
-					(size 1.27 1.27)
-				)
-				(hide yes)
-			)
-		)
-		(pin "2"
-		)
-		(pin "1"
-		)
-		(instances
-			(project ""
-				(path "/5d40675e-f021-4f7d-ab90-3f579d2e0ed7"
-					(reference "D1")
-					(unit 1)
-				)
-			)
-		)
-	)
-	(symbol
 		(lib_id "power:VCC")
 		(at 46.99 73.66 0)
@@
 					(unit 1)
 				)
-			)
-		)
-	)
-	(symbol
-		(lib_id "power:GND")
-		(at 50.8 40.64 0)
-		(unit 1)
-		(exclude_from_sim no)
-		(in_bom yes)
-		(on_board yes)
-		(dnp no)
-		(fields_autoplaced yes)
-		(property "Reference" "#PWR04"
-			(at 50.8 46.99 0)
-			(effects
-				(font
-					(size 1.27 1.27)
-				)
-				(hide yes)
-			)
-		)
-		(property "Value" "GND"
-			(at 50.8 45.72 0)
-			(effects
-				(font
-					(size 1.27 1.27)
-				)
-			)
-		)
-		(property "Footprint" ""
-			(at 50.8 40.64 0)
-			(effects
-				(font
-					(size 1.27 1.27)
-				)
-				(hide yes)
-			)
-		)
-		(property "Datasheet" ""
-			(at 50.8 40.64 0)
-			(effects
-				(font
-					(size 1.27 1.27)
-				)
-				(hide yes)
-			)
-		)
-		(property "Description" "Power symbol creates a global label with name \"GND\" , ground"
-			(at 50.8 40.64 0)
-			(effects
-				(font
-					(size 1.27 1.27)
-				)
-				(hide yes)
-			)
-		)
-		(pin "1"
-		)
-		(instances
-			(project "CardPCB"
-				(path "/5d40675e-f021-4f7d-ab90-3f579d2e0ed7"
-					(reference "#PWR04")
-					(unit 1)
-				)

Commit message: Dossier de remise
voila
Other:
- note added: "*2 BT2 is for external power"
- note removed: "*2 Right source is for testing purposes only"
- moved on the sheet: D6, H1, H2, Q1, R3, R4
